File: MotherClock/MotherClock.kicad_pcb (KiCad board)
At the start: 2 copper layers, 80 x 85 mm, 58 parts, among them J1 Main, J2 DS3231 Module, J3 OLED, J4 LED, Q1 BC856, Q2 BC846, Q3 BC856, Q4 BC846, Q5 BC556, Q6 BC546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

Commit message: Update PCB to KiCad 6
Other:
- net class Default removed
